File: viaems/viaems.kicad_pcb (KiCad board)
At the start: 2 copper layers, 207 parts, among them J1 Conn_02x08_Counter_Clockwise, J10 Conn_01x04, J11 Conn_01x08, J12 Conn_01x02, J13 Conn_01x06, J14 Conn_01x06, J15 Conn_02x06_Odd_Even, J16 VBAT, J17 Conn_01x04, J18 USB_B_Micro, J19 Conn_ARM_JTAG_SWD_10, J2 Conn_01x02, J20 SPI, J3 Conn_01x03, J4 Conn_01x04, J5 Conn_01x02, J6 Conn_01x02, J7 Conn_01x06, J8 Conn_01x04, J9 Conn_01x08, Q1 VND7NV04, Q2 VND7NV04, Q3 VND7NV04, Q4 VND7NV04, Q5 VND7NV04, Q6 VND7NV04, Q7 VND7NV04, Q8 VND7NV04, U1 LM2940, U10 MCP2562-H-SN, U11 NCP1117-3.3_TO252, U12 MPXH6400A, U13 MPXH6115AC6U, U14 MAX9926UAEE+, U15 LM2940, U16 AD7888, U2 TC442xA, U3 TC442xA, U4 TC442xA, U5 TC442xA, U6 TC442xA, U7 TC442xA, U8 TC442xA, U9 STM32F407VGTx, Y1 8 Mhz

Commit message: More routing
Parts:
- C11, C13, C16, C26: moved to B.Cu
- C15, C19, C21, C22, C24: value 100 nF -> 0.1 uF; moved to B.Cu
- C18, C20, C23: value 100 nF -> 0.1 uF
- moved J2 165.3 mm to (83.2, 111.1), turned to 180 degrees
- moved J6 85.1 mm to (122.6, 102.9), turned to 270 degrees
- moved J9 84.4 mm to (153.7, 81.3)
- moved J17 78.2 mm to (131.4, 97.2), turned to 180 degrees
- moved C23 70.2 mm to (168.9, 69.9)
- moved R50 58.5 mm to (113.7, 130.8), turned to 90 degrees
- moved C11 45.7 mm to (129.5, 85.1), turned to 0 degrees
- moved C13 41.1 mm to (124.5, 85.1)
- moved Y1 40.8 mm to (129.6, 82.6), turned to 180 degrees
- moved R48 40.0 mm to (80.6, 88.9), turned to 0 degrees
- moved J8 38.6 mm to (91.4, 100.3), turned to 90 degrees
- moved J3 32.5 mm to (106.0, 80.6)
- moved R2 32.2 mm to (87.6, 100.3), turned to 180 degrees
- moved R1 30.7 mm to (87.6, 102.9), turned to 180 degrees
- moved C26 29.5 mm to (119.4, 85.1), turned to 225 degrees
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Connections:
- C54 pad 1: Net-(C54-Pad1) -> 5v_cpu
- C56 pad 1: Net-(C54-Pad1) -> 5v_cpu
- C57 pad 1: Net-(C54-Pad1) -> 5v_cpu
- D3 pad 2: /Inputs/5v_analog -> 5v_cpu
- D8 pad 2: /Inputs/5v_analog -> 5v_cpu
- J1 pad 1: GND -> /Inputs/IN1-
- J1 pad 14: /Inputs/SPR1 -> /Inputs/EGO
- J1 pad 2: GND -> /Inputs/IN2+
- J1 pad 3: /Inputs/IN1- -> /Inputs/IN1+
- J1 pad 4: /Inputs/IN1+ -> /Inputs/IN2-
- J1 pad 5: /Inputs/IN2- -> /Inputs/DIG2
- J1 pad 6: /Inputs/IN2+ -> /Inputs/DIG1
- J1 pad 7: /Inputs/DIG2 -> GND
- J1 pad 8: /Inputs/DIG1 -> GND
- J1 pad 9: /Inputs/EGO -> /Inputs/SPR1
- J15 pad 1: /Outputs/IG1-out -> /Outputs/HSD1-out
- J15 pad 10: /Outputs/12v_output -> /CANL
- J15 pad 11: /Outputs/HSD2-out -> /12v_switched
- J15 pad 2: /12v_switched -> /Outputs/IG4-out
- J15 pad 3: /Outputs/IG2-out -> /Outputs/12v_output
- J15 pad 4: /CANH -> /Outputs/IG3-out
- J15 pad 5: /Outputs/IG3-out -> /Outputs/12v_output
- J15 pad 6: /CANL -> /Outputs/IG2-out
- J15 pad 7: /Outputs/IG4-out -> /Outputs/HSD2-out
- J15 pad 8: /Outputs/12v_output -> /Outputs/IG1-out
- J15 pad 9: /Outputs/HSD1-out -> /CANH
- J19 pad 6: (no net) -> Net-(J19-Pad6)
- J19 pad 7: (no net) -> Net-(J19-Pad7)
- J19 pad 8: (no net) -> Net-(J19-Pad8)
- J20 pad 2: /Cpu/SCK-cpu -> /Inputs/CS
- J20 pad 3: /Inputs/MOSI -> /Cpu/SCK-cpu
- J20 pad 4: /Inputs/CS -> /Inputs/MISO
- J20 pad 5: /Inputs/MISO -> /Inputs/MOSI
- J20 pad 6: /Inputs/5v_analog -> 5v_cpu
- R70 pad 1: /Inputs/5v_analog -> 5v_cpu
- R71 pad 1: /Inputs/5v_analog -> 5v_cpu
- U12 pad 1: (no net) -> Net-(U12-Pad1)
- U12 pad 5: (no net) -> Net-(U12-Pad5)
- U12 pad 6: (no net) -> Net-(U12-Pad6)
- U12 pad 7: (no net) -> Net-(U12-Pad7)
- U12 pad 8: (no net) -> Net-(U12-Pad8)
- U13 pad 1: (no net) -> Net-(U13-Pad1)
- U13 pad 5: (no net) -> Net-(U13-Pad5)
- U13 pad 6: (no net) -> Net-(U13-Pad6)
- U13 pad 7: (no net) -> Net-(U13-Pad7)
- U13 pad 8: (no net) -> Net-(U13-Pad8)
- U14 pad 12: (no net) -> Net-(U14-Pad12)
- U14 pad 14: Net-(C54-Pad1) -> 5v_cpu
- U14 pad 2: (no net) -> Net-(U14-Pad2)
- U14 pad 7: (no net) -> Net-(U14-Pad7)
- U2 pad 1: (no net) -> Net-(U2-Pad1)
- U2 pad 8: (no net) -> Net-(U2-Pad8)
- U3 pad 1: (no net) -> Net-(U3-Pad1)
- U3 pad 8: (no net) -> Net-(U3-Pad8)
- U4 pad 1: (no net) -> Net-(U4-Pad1)
- U4 pad 8: (no net) -> Net-(U4-Pad8)
- U5 pad 1: (no net) -> Net-(U5-Pad1)
- U5 pad 8: (no net) -> Net-(U5-Pad8)
- U6 pad 1: (no net) -> Net-(U6-Pad1)
- U6 pad 8: (no net) -> Net-(U6-Pad8)
- U7 pad 1: (no net) -> Net-(U7-Pad1)
- U7 pad 8: (no net) -> Net-(U7-Pad8)
- U8 pad 1: (no net) -> Net-(U8-Pad1)
- U8 pad 8: (no net) -> Net-(U8-Pad8)
- U9 pad 15: (no net) -> Net-(U9-Pad15)
- U9 pad 16: (no net) -> Net-(U9-Pad16)
- U9 pad 17: (no net) -> Net-(U9-Pad17)
- U9 pad 18: (no net) -> Net-(U9-Pad18)
- U9 pad 26: (no net) -> Net-(U9-Pad26)
- U9 pad 29: (no net) -> Net-(U9-Pad29)
- U9 pad 30: (no net) -> Net-(U9-Pad30)
- U9 pad 31: (no net) -> Net-(U9-Pad31)
- U9 pad 32: (no net) -> Net-(U9-Pad32)
- U9 pad 33: (no net) -> Net-(U9-Pad33)
- U9 pad 34: (no net) -> Net-(U9-Pad34)
- U9 pad 35: (no net) -> Net-(U9-Pad35)
- U9 pad 36: (no net) -> Net-(U9-Pad36)
- U9 pad 39: (no net) -> Net-(U9-Pad39)
- U9 pad 40: (no net) -> Net-(U9-Pad40)
- U9 pad 41: (no net) -> Net-(U9-Pad41)
- U9 pad 42: (no net) -> Net-(U9-Pad42)
- U9 pad 43: (no net) -> Net-(U9-Pad43)
- U9 pad 44: (no net) -> Net-(U9-Pad44)
- U9 pad 45: (no net) -> Net-(U9-Pad45)
- U9 pad 46: (no net) -> Net-(U9-Pad46)
- U9 pad 48: (no net) -> Net-(U9-Pad48)
- U9 pad 67: (no net) -> Net-(U9-Pad67)
- U9 pad 77: (no net) -> Net-(U9-Pad77)
- U9 pad 8: (no net) -> Net-(U9-Pad8)
- U9 pad 9: (no net) -> Net-(U9-Pad9)
- U9 pad 90: (no net) -> Net-(U9-Pad90)
- U9 pad 93: (no net) -> Net-(U9-Pad93)
Routing:
- net /Inputs/5v_analog: track 0.00 -> 229.2 mm, vias 0 -> 2
- net 5v_cpu: track 63.1 -> 266.0 mm, vias 0 -> 5
- net GND: track 71.1 -> 203.5 mm, vias 14 -> 63
- net /Cpu/3v_cpu: track 0.00 -> 106.6 mm, vias 0 -> 4
- net /Cpu/GPIO1-cpu: track 0.00 -> 47.8 mm, vias 0 -> 2
- net /CANL: track 0.00 -> 47.6 mm
- net /CANH: track 0.00 -> 46.3 mm
- net /Cpu/GPIO2-cpu: track 0.00 -> 40.6 mm, vias 0 -> 2
- net /Inputs/CS: track 0.00 -> 40.6 mm
- net /Cpu/USB-DM: track 0.00 -> 37.6 mm, vias 0 -> 2
- net /Cpu/USB-DP: track 0.00 -> 37.2 mm, vias 0 -> 2
- net /Cpu/SCK-cpu: track 0.00 -> 36.4 mm
- net /Cpu/USB-ID: track 0.00 -> 34.0 mm, vias 0 -> 2
- net /Inputs/MISO: track 0.00 -> 33.9 mm
- net /Cpu/GPIO3-cpu: track 0.00 -> 32.9 mm
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- added copper zone on F.Cu, net /Cpu/3v_cpu
- added copper zone on B.Cu, net GND

Commit message: Finished routing
Parts:
- added J21: Conn_01x02, Connector_PinHeader_2.54mm:PinHeader_1x02_P2.54mm_Vertical, F.Cu at (92.7, 95.2)
- added REF**: SolderWirePad_1x01_Drill2.5mm, Connector_Wire:SolderWirePad_1x01_Drill2.5mm, F.Cu at (166.4, 83.8)
- added REF**: SolderWirePad_1x01_Drill2.5mm, Connector_Wire:SolderWirePad_1x01_Drill2.5mm, F.Cu at (47.0, 83.8)
- C19, C24, C26: moved to F.Cu
- C20, C23, D1, J18, R46, R48, R51, R52, R53: moved to B.Cu
- J7: value Conn_01x06 -> Conn_01x04; footprint Connector_PinHeader_2.54mm:PinHeader_1x06_P2.54mm_Vertical -> Connector_PinHeader_2.54mm:PinHeader_1x04_P2.54mm_Vertical
- moved J7 103.6 mm to (97.8, 114.3), turned to 0 degrees
- moved C30 74.5 mm to (154.3, 82.5)
- moved U11 71.0 mm to (159.4, 85.1)
- moved C29 66.6 mm to (152.4, 86.4), turned to 90 degrees
- moved C23 59.3 mm to (116.2, 97.0), turned to 90 degrees
- moved C27 51.5 mm to (121.3, 104.1), turned to 270 degrees
- moved C28 51.3 mm to (118.7, 104.1), turned to 270 degrees
- moved JP1 49.9 mm to (110.5, 108.0), turned to 270 degrees
- moved R45 47.9 mm to (111.1, 104.8), turned to 90 degrees
- moved R46 46.2 mm to (111.1, 102.2), turned to 0 degrees
- moved J16 42.9 mm to (125.7, 100.3), turned to 90 degrees
- moved D1 42.6 mm to (123.8, 97.8), turned to 270 degrees
- moved J17 41.2 mm to (94.0, 114.3), turned to 0 degrees
- moved J9 37.4 mm to (132.1, 111.8), turned to 180 degrees
- moved R84 31.0 mm to (148.1, 86.0)
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Connections:
- net /Cpu/BOOT renamed Net-(JP1-Pad2)
- JP1 pad 1: 5v_cpu -> /Cpu/3v_cpu
Routing:
- net /Cpu/3v_cpu: track 106.6 -> 176.6 mm, vias 4 -> 29
- net GND: track 203.5 -> 271.1 mm, vias 63 -> 74
- net Net-(R85-Pad2): track 0.00 -> 62.0 mm, vias 0 -> 2
- net Net-(R84-Pad2): track 0.00 -> 60.8 mm
- net /Cpu/TRIG1-cpu: track 6.99 -> 51.3 mm
- net /Cpu/TRIG2-cpu: track 3.93 -> 47.1 mm, vias 0 -> 2
- net Net-(J17-Pad4): track 14.5 -> 46.1 mm, vias 2 -> 0
- net /Cpu/NRST: track 0.00 -> 28.7 mm
- net /Cpu/GPIO8-cpu: track 0.00 -> 28.0 mm, vias 0 -> 2
- net /Cpu/OUT4-cpu: track 0.00 -> 27.5 mm
- net /Cpu/OUT3-cpu: track 0.00 -> 24.8 mm
- net /Cpu/USB-DM: track 37.6 -> 14.2 mm, vias 2 -> 1
- net /Cpu/GPIO1-cpu: track 47.8 -> 24.7 mm, vias 2 -> 0
- net 5v_cpu: track 266.0 -> 243.2 mm
- net /Cpu/USB-DP: track 37.2 -> 14.4 mm, vias 2 -> 1
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- added copper zone on B.Cu, net /Cpu/3v_cpu
Other:
- board outline added: 136 x 64 mm
