File: viaems/viaems.sch (KiCad schematic (older format))
At the start: 20 parts, among them J1 Conn_02x06_Counter_Clockwise, J10 Conn_01x06, J11 Conn_01x02, J12 Conn_01x06, J13 Conn_01x06, J14 Conn_02x06_Counter_Clockwise, J2 Conn_01x02, J3 Conn_01x03, J4 Conn_01x04, J5 Conn_01x02, J6 Conn_01x06, J7 Conn_01x04, J8 Conn_01x08, J9 Conn_01x06, U1 LM2940

Commit message: More progress. Calling schematic complete, board partially routed
Parts:
- removed J1: Conn_02x06_Counter_Clockwise, symbol Connector_Generic:Conn_02x06_Counter_Clockwise
- added J1: Conn_02x08_Counter_Clockwise, Connector_PinHeader_2.54mm:PinHeader_2x08_P2.54mm_Vertical, symbol Connector_Generic:Conn_02x08_Counter_Clockwise
- added J5: Conn_01x02, Connector_PinHeader_2.54mm:PinHeader_1x02_P2.54mm_Vertical, symbol Connector_Generic:Conn_01x02
- added R1, R2, R3, R4: 100k, Resistor_SMD:R_0805_2012Metric_Pad1.15x1.40mm_HandSolder, symbol Device:R
- C1: footprint (none) -> Capacitor_SMD:C_1206_3216Metric_Pad1.42x1.75mm_HandSolder; Digikey-Part (none) -> 445-14799-1-ND; Notes (none) -> 35V
- C2, C3: footprint (none) -> Capacitor_SMD:C_0805_2012Metric_Pad1.15x1.40mm_HandSolder
- C4: footprint (none) -> Capacitor_SMD:C_1206_3216Metric_Pad1.42x1.75mm_HandSolder; Digikey-Part (none) -> 478-9009-1-ND; Notes (none) -> Tantalum
- J10: renamed from J9; value Conn_01x06 -> Conn_01x04; footprint (none) -> Connector_PinHeader_2.54mm:PinHeader_1x04_P2.54mm_Vertical; symbol Connector_Generic:Conn_01x06 -> Connector_Generic:Conn_01x04
- J11: renamed from J10; value Conn_01x06 -> Conn_01x08; footprint (none) -> Connector_PinHeader_2.54mm:PinHeader_1x08_P2.54mm_Vertical; symbol Connector_Generic:Conn_01x06 -> Connector_Generic:Conn_01x08
- J12: renamed from J11; footprint (none) -> Connector_PinHeader_2.54mm:PinHeader_1x02_P2.54mm_Vertical
- J13: renamed from J12; footprint (none) -> Connector_PinHeader_2.54mm:PinHeader_1x06_P2.54mm_Vertical
- J14: renamed from J13; footprint (none) -> Connector_PinHeader_2.54mm:PinHeader_1x06_P2.54mm_Vertical
- J15: renamed from J14; value Conn_02x06_Counter_Clockwise -> Conn_02x06_Odd_Even; footprint (none) -> Connector_PinHeader_2.54mm:PinHeader_2x06_P2.54mm_Vertical; symbol Connector_Generic:Conn_02x06_Counter_Clockwise -> Connector_Generic:Conn_02x06_Odd_Even
- J2, JP1: footprint (none) -> Connector_PinHeader_2.54mm:PinHeader_1x02_P2.54mm_Vertical
- J3: footprint (none) -> Connector_PinHeader_2.54mm:PinHeader_1x03_P2.54mm_Vertical
- J4: footprint (none) -> Connector_PinHeader_2.54mm:PinHeader_1x04_P2.54mm_Vertical
- J6: renamed from J5; footprint (none) -> Connector_PinHeader_2.54mm:PinHeader_1x02_P2.54mm_Vertical
- J7: renamed from J6; footprint (none) -> Connector_PinHeader_2.54mm:PinHeader_1x06_P2.54mm_Vertical
- J8: renamed from J7; footprint (none) -> Connector_PinHeader_2.54mm:PinHeader_1x04_P2.54mm_Vertical
- J9: renamed from J8; footprint (none) -> Connector_PinHeader_2.54mm:PinHeader_1x08_P2.54mm_Vertical
- U1: footprint (none) -> Package_TO_SOT_THT:TO-220-3_Horizontal_TabDown
Connections:
- net 12v_switched: now also J15.2 (Pin_2); no longer J15.6 (Pin_6)
- net 5v_cpu: now also R1.2, R2.2, R3.2, R4.2
- net Cpu/CS-cpu: now also R4.1
- net Cpu/INJ1-cpu: now also J11.8 (Pin_8); no longer J10.5 (Pin_5)
- net Cpu/INJ2-cpu: now also J11.7 (Pin_7); no longer J10.6 (Pin_6)
- net Cpu/MISO-cpu: now also R2.1
- net Cpu/MOSI-cpu: now also R1.1
- net Cpu/SCK-cpu: now also R3.1
- net Cpu/TRIG1-cpu: now also J5.2 (Pin_2)
- net Cpu/TRIG2-cpu: now also J5.1 (Pin_1)
- net GND: now also J15.12 (Pin_12); no longer J15.1 (Pin_1)
- net Inputs/12v_analog: now also J1.16 (Pin_16)
- net Inputs/5v_out: now also J1.15 (Pin_15)
- net Inputs/BRV: now also J1.11 (Pin_11)
- net Inputs/CLT: now also J1.13 (Pin_13)
- net Inputs/DIG1: now also J1.8 (Pin_8)
- net Inputs/DIG2: now also J1.7 (Pin_7)
- net Inputs/EGO: now also J1.9 (Pin_9)
- net Inputs/IAT: now also J1.12 (Pin_12)
- net Inputs/SENSOR_GND: now also J1.1 (Pin_1), J1.2 (Pin_2)
- net Inputs/SPR1: now also J1.14 (Pin_14)
- net Inputs/TPS: now also J1.10 (Pin_10)
- net Outputs/12v_output: now also J15.10 (Pin_10), J15.8 (Pin_8); no longer J15.2 (Pin_2), J15.3 (Pin_3)
- net Outputs/HSD1-out: now also J15.9 (Pin_9); no longer J15.11 (Pin_11)
- net Outputs/HSD2-out: now also J15.11 (Pin_11); no longer J15.12 (Pin_12)
- net Outputs/IG1-out: now also J15.1 (Pin_1); no longer J15.7 (Pin_7)
- net Outputs/IG2-out: now also J15.3 (Pin_3); no longer J15.8 (Pin_8)
- net Outputs/IG3-out: now also J15.5 (Pin_5); no longer J15.9 (Pin_9)
- net Outputs/IG4-out: now also J15.7 (Pin_7); no longer J15.10 (Pin_10)
- net CANH: now reaches J15.4 (Pin_4)
- new net CANL: J15.6 (Pin_6)
- new net Inputs/IN1+: J1.4 (Pin_4)
- new net Inputs/IN1-: J1.3 (Pin_3)
- new net Inputs/IN2+: J1.6 (Pin_6)
- new net Inputs/IN2-: J1.5 (Pin_5)
- no-connect marks 2 -> 0
Other:
- moved on the sheet: J12, J13, J14, J15, J2, J3, J4, J6, J7, J8, J9, JP1

Commit message: More routing
Connections:
- net 12v_switched: now also J15.11 (Pin_11); no longer J15.2 (Pin_2)
- net CANH: now also J15.9 (Pin_9); no longer J15.4 (Pin_4)
- net CANL: now also J15.10 (Pin_10); no longer J15.6 (Pin_6)
- net Inputs/DIG1: now also J1.6 (Pin_6); no longer J1.8 (Pin_8)
- net Inputs/DIG2: now also J1.5 (Pin_5); no longer J1.7 (Pin_7)
- net Inputs/EGO: now also J1.14 (Pin_14); no longer J1.9 (Pin_9)
- net Inputs/IN1+: now also J1.3 (Pin_3); no longer J1.4 (Pin_4)
- net Inputs/IN1-: now also J1.1 (Pin_1); no longer J1.3 (Pin_3)
- net Inputs/IN2+: now also J1.2 (Pin_2); no longer J1.6 (Pin_6)
- net Inputs/IN2-: now also J1.4 (Pin_4); no longer J1.5 (Pin_5)
- net Inputs/SENSOR_GND: now also J1.7 (Pin_7), J1.8 (Pin_8); no longer J1.1 (Pin_1), J1.2 (Pin_2)
- net Inputs/SPR1: now also J1.9 (Pin_9); no longer J1.14 (Pin_14)
- net Outputs/12v_output: now also J15.3 (Pin_3), J15.5 (Pin_5); no longer J15.10 (Pin_10), J15.8 (Pin_8)
- net Outputs/HSD1-out: now also J15.1 (Pin_1); no longer J15.9 (Pin_9)
- net Outputs/HSD2-out: now also J15.7 (Pin_7); no longer J15.11 (Pin_11)
- net Outputs/IG1-out: now also J15.8 (Pin_8); no longer J15.1 (Pin_1)
- net Outputs/IG2-out: now also J15.6 (Pin_6); no longer J15.3 (Pin_3)
- net Outputs/IG3-out: now also J15.4 (Pin_4); no longer J15.5 (Pin_5)
- net Outputs/IG4-out: now also J15.2 (Pin_2); no longer J15.7 (Pin_7)
Other:
- moved on the sheet: J15
Changed lines of the file:
@@
 F23 "IN1-" I L 2350 5650 50
 F24 "IN1+" I L 2350 5550 50
+F25 "5v_cpu" I R 3750 4250 50
 $EndSheet
 Wire Wire Line
@@
 L Connector_Generic:Conn_02x06_Odd_Even J15
 U 1 1 5C10B27C
-P 10300 4100
-F 0 "J15" H 10350 3667 50  0000 C CNN
-F 1 "Conn_02x06_Odd_Even" H 10350 4426 50  0001 C CNN
-F 2 "Connector_PinHeader_2.54mm:PinHeader_2x06_P2.54mm_Vertical" H 10300 4100 50  0001 C CNN
-F 3 "~" H 10300 4100 50  0001 C CNN
-	1    10300 4100
-	1    0    0    -1
-$EndComp
-Wire Wire Line
-	9450 3900 10100 3900
-Wire Wire Line
-	9450 4000 10100 4000
-Wire Wire Line
-	9450 4100 10100 4100
-Wire Wire Line
-	9450 4200 10100 4200
-Wire Wire Line
-	9450 4300 10100 4300
-Wire Wire Line
-	9450 4400 10100 4400
+P 10500 4250
+F 0 "J15" H 10550 4550 50  0000 C CNN
+F 1 "Conn_02x06_Odd_Even" H 10550 4576 50  0001 C CNN
+F 2 "Connector_PinHeader_2.54mm:PinHeader_2x06_P2.54mm_Vertical" H 10500 4250 50  0001 C CNN
+F 3 "~" H 10500 4250 50  0001 C CNN
+	1    10500 4250
+	1    0    0    -1
+$EndComp
 $Comp
 L power:GND #PWR06
 U 1 1 5C153578
-P 10600 4400
-F 0 "#PWR06" H 10600 4150 50  0001 C CNN
-F 1 "GND" H 10605 4227 50  0001 C CNN
-F 2 "" H 10600 4400 50  0001 C CNN
-F 3 "" H 10600 4400 50  0001 C CNN
-	1    10600 4400
-	1    0    0    -1
-$EndComp
-Wire Wire Line
-	9450 4550 10650 4550
-Wire Wire Line
-	10650 4550 10650 4300
-Wire Wire Line
-	10650 4300 10600 4300
-Text Label 10600 3900 0    50   ~ 0
+P 10800 4550
+F 0 "#PWR06" H 10800 4300 50  0001 C CNN
+F 1 "GND" H 10805 4377 50  0001 C CNN
+F 2 "" H 10800 4550 50  0001 C CNN
+F 3 "" H 10800 4550 50  0001 C CNN
+	1    10800 4550
+	1    0    0    -1
+$EndComp
+Text Label 10300 4550 2    50   ~ 0
 12v_switched
 $Comp
@@
 	10050 5700 10100 5700
 Connection ~ 10050 5400
-Wire Wire Line
-	10650 4300 10650 4200
-Wire Wire Line
-	10650 4200 10600 4200
-Connection ~ 10650 4300
 $Comp
 L Device:R R?
@@
 L power:PWR_FLAG #FLG02
 U 1 1 5C0F8D45
-P 10650 4300
-F 0 "#FLG02" H 10650 4375 50  0001 C CNN
-F 1 "PWR_FLAG" V 10650 4428 50  0000 L CNN
-F 2 "" H 10650 4300 50  0001 C CNN
-F 3 "~" H 10650 4300 50  0001 C CNN
-	1    10650 4300
-	0    1    1    0
+P 10150 4150
+F 0 "#FLG02" H 10150 4225 50  0001 C CNN
+F 1 "PWR_FLAG" H 10150 4250 50  0001 L CNN
+F 2 "" H 10150 4150 50  0001 C CNN
+F 3 "~" H 10150 4150 50  0001 C CNN
+	1    10150 4150
+	1    0    0    -1
 $EndComp
 $Comp
@@
 	1750 4250 2350 4250
 Wire Wire Line
-	1800 4350 1800 4600
-Wire Wire Line
-	1800 4600 1650 4600
-Wire Wire Line
-	1650 4700 1850 4700
-Wire Wire Line
-	1850 4700 1850 4450
-Wire Wire Line
-	1850 4450 2350 4450
-Wire Wire Line
-	2350 4550 1900 4550
-Wire Wire Line
-	1900 4550 1900 4800
-Wire Wire Line
-	1900 4800 1650 4800
-Wire Wire Line
-	2350 4650 1950 4650
-Wire Wire Line
-	1950 4650 1950 4900
-Wire Wire Line
-	1950 4900 1650 4900
-Wire Wire Line
-	2350 4750 2000 4750
-Wire Wire Line
-	2000 4750 2000 5000
-Wire Wire Line
-	2000 5000 1650 5000
-Wire Wire Line
-	1650 5100 2050 5100
-Wire Wire Line
-	2050 5100 2050 4850
-Wire Wire Line
-	2050 4850 2350 4850
-Wire Wire Line
 	2350 4950 2100 4950
 Wire Wire Line
@@
 	2100 5250 1100 5250
 Wire Wire Line
-	1100 5250 1100 5100
-Wire Wire Line
-	1100 5100 1150 5100
-Wire Wire Line
 	2350 5050 2150 5050
 Wire Wire Line
@@
 	2150 5300 1050 5300
 Wire Wire Line
-	1050 5300 1050 5000
-Wire Wire Line
-	1050 5000 1150 5000
-Wire Wire Line
 	2350 5350 1000 5350
 Wire Wire Line
-	1000 5350 1000 4900
-Wire Wire Line
-	1000 4900 1150 4900
-Wire Wire Line
 	2350 5450 950  5450
 Wire Wire Line
-	950  5450 950  4800
-Wire Wire Line
-	950  4800 1150 4800
-Wire Wire Line
 	2350 5550 900  5550
 Wire Wire Line
-	900  5550 900  4700
-Wire Wire Line
-	900  4700 1150 4700
-Wire Wire Line
 	2350 5650 850  5650
-Wire Wire Line
-	850  5650 850  4600
-Wire Wire Line
-	850  4600 1150 4600
-Wire Wire Line
-	2350 5850 800  5850
-Wire Wire Line
-	800  5850 800  4500
-Wire Wire Line
-	800  4500 1050 4500
-Wire Wire Line
-	1150 4400 1050 4400
-Wire Wire Line
-	1050 4400 1050 4500
-Connection ~ 1050 4500
-Wire Wire Line
-	1050 4500 1150 4500
 $Comp
 L Connector_Generic:Conn_01x02 J5
@@
 Wire Wire Line
 	3750 5100 4600 5100
-Text Label 10600 4000 0    50   ~ 0
+Text Label 10300 4450 2    50   ~ 0
 CANH
-Text Label 10600 4100 0    50   ~ 0
+Text Label 10800 4450 0    50   ~ 0
 CANL
 Text Label 6400 6300 0    50   ~ 0
@@
 	6250 6400 6400 6400
 Wire Wire Line
-	1800 4350 2350 4350
-Wire Wire Line
 	6250 4200 7550 4200
 Wire Wire Line
@@
 	7400 4650 7650 4650
 Connection ~ 7650 4650
+Wire Wire Line
+	4250 4050 4250 4250
+Wire Wire Line
+	4250 4250 3750 4250
+Wire Wire Line
+	10300 4350 10000 4350
+Wire Wire Line
+	10000 4350 10000 4400
+Wire Wire Line
+	10000 4400 9450 4400
+Wire Wire Line
+	9450 4300 10250 4300
+Wire Wire Line
+	10250 4300 10250 4050
+Wire Wire Line
+	10250 4050 10300 4050
+Wire Wire Line
+	9450 4550 9800 4550
+Wire Wire Line
+	9800 4550 9800 4250
+Wire Wire Line
+	9800 4250 10150 4250
+Wire Wire Line
+	10150 4250 10150 4150
+Wire Wire Line
+	10150 4150 10300 4150
+Connection ~ 10150 4250
+Wire Wire Line
+	10150 4250 10300 4250
+Wire Wire Line
+	9450 4200 10100 4200
+Wire Wire Line
+	10100 4200 10100 3900
+Wire Wire Line
+	10100 3900 10850 3900
+Wire Wire Line
+	10850 3900 10850 4050
+Wire Wire Line
+	10850 4050 10800 4050
+Wire Wire Line
+	9450 4100 10050 4100
+Wire Wire Line
+	10050 4100 10050 3850
+Wire Wire Line
+	10050 3850 10900 3850
+Wire Wire Line
+	10900 3850 10900 4150
+Wire Wire Line
+	10900 4150 10800 4150
+Wire Wire Line
+	10800 4250 10950 4250
+Wire Wire Line
+	10950 4250 10950 3800
+Wire Wire Line
+	10950 3800 10000 3800
+Wire Wire Line
+	10000 3800 10000 4000
+Wire Wire Line
+	10000 4000 9450 4000
+Wire Wire Line
+	9450 3900 9950 3900
+Wire Wire Line
+	9950 3900 9950 3750
+Wire Wire Line
+	9950 3750 11000 3750
+Wire Wire Line
+	11000 3750 11000 4350
+Wire Wire Line
+	11000 4350 10800 4350
+Connection ~ 10150 4150
+Wire Wire Line
+	850  5650 850  4400
+Wire Wire Line
+	850  4400 1150 4400
+Wire Wire Line
+	900  5550 900  4600
+Wire Wire Line
+	900  4600 1150 4600
+Wire Wire Line
+	1000 5350 1000 4500
+Wire Wire Line
+	1000 4500 1150 4500
+Wire Wire Line
+	950  5450 950  4700
+Wire Wire Line
+	950  4700 1150 4700
+Wire Wire Line
+	1100 5250 1100 4900
+Wire Wire Line
+	1100 4900 1150 4900
+Wire Wire Line
+	1050 5300 1050 4800
+Wire Wire Line
+	1050 4800 1150 4800
+Wire Wire Line
+	2350 5850 1150 5850
+Wire Wire Line
+	1150 5850 1150 5100
+Wire Wire Line
+	1150 5100 1150 5000
+Connection ~ 1150 5100
+Wire Wire Line
+	2350 4850 2200 4850
+Wire Wire Line
+	2200 4850 2200 4600
+Wire Wire Line
+	2200 4600 1650 4600
+Wire Wire Line
+	2350 4450 1800 4450
+Wire Wire Line
+	1800 4450 1800 4700
+Wire Wire Line
+	1800 4700 1650 4700
+Wire Wire Line
+	2350 4550 1850 4550
+Wire Wire Line
+	1850 4550 1850 4800
+Wire Wire Line
+	1850 4800 1650 4800
+Wire Wire Line
+	2350 4650 1900 4650
+Wire Wire Line
+	1900 4650 1900 4900
+Wire Wire Line
+	1900 4900 1650 4900
+Wire Wire Line
+	2350 4750 1950 4750
+Wire Wire Line
+	1950 4750 1950 5000
+Wire Wire Line
+	1950 5000 1650 5000
+Wire Wire Line
+	2350 4350 2000 4350
+Wire Wire Line
+	2000 4350 2000 5100
+Wire Wire Line
+	2000 5100 1650 5100
 $EndSCHEMATC

Commit message: Finished routing
Parts:
- removed J7: Conn_01x06, Connector_PinHeader_2.54mm:PinHeader_1x06_P2.54mm_Vertical, symbol Connector_Generic:Conn_01x06
- removed JP1: Jumper, Connector_PinHeader_2.54mm:PinHeader_1x02_P2.54mm_Vertical, symbol Device:Jumper
- added J21: Conn_01x02, Connector_PinHeader_2.54mm:PinHeader_1x02_P2.54mm_Vertical, symbol Connector_Generic:Conn_01x02
- added J7: Conn_01x04, Connector_PinHeader_2.54mm:PinHeader_1x04_P2.54mm_Vertical, symbol Connector_Generic:Conn_01x04
Connections:
- net Cpu/OUT1-cpu: now also J7.1 (Pin_1)
- net Cpu/OUT2-cpu: now also J7.2 (Pin_2)
- net Cpu/OUT3-cpu: now also J7.3 (Pin_3)
- net Cpu/OUT4-cpu: now also J7.4 (Pin_4)
- net Cpu/OUT5-cpu: now also J21.1 (Pin_1)
- net Cpu/OUT6-cpu: now also J21.2 (Pin_2)
Changed lines of the file:
@@
 F0 "Cpu" 50
 F1 "cpu.sch" 50
-F2 "BOOT" I L 4950 3750 50
-F3 "IG1-cpu" I R 6250 3700 50
-F4 "IG2-cpu" I R 6250 3800 50
-F5 "IG3-cpu" I R 6250 3900 50
-F6 "IG4-cpu" I R 6250 4000 50
-F7 "INJ1-cpu" I R 6250 4100 50
-F8 "INJ2-cpu" I R 6250 4200 50
-F9 "INJ3-cpu" I R 6250 4300 50
-F10 "INJ4-cpu" I R 6250 4400 50
-F11 "INJ5-cpu" I R 6250 4500 50
-F12 "INJ6-cpu" I R 6250 4600 50
-F13 "OUT1-cpu" I R 6250 4700 50
-F14 "OUT2-cpu" I R 6250 4800 50
-F15 "OUT3-cpu" I R 6250 4900 50
-F16 "OUT4-cpu" I R 6250 5000 50
-F17 "OUT5-cpu" I R 6250 5100 50
-F18 "OUT6-cpu" I R 6250 5200 50
-F19 "GPIO1-cpu" I R 6250 5300 50
-F20 "GPIO2-cpu" I R 6250 5400 50
-F21 "GPIO3-cpu" I R 6250 5500 50
-F22 "GPIO4-cpu" I R 6250 5600 50
-F23 "GPIO5-cpu" I R 6250 5700 50
-F24 "GPIO6-cpu" I R 6250 5800 50
-F25 "GPIO7-cpu" I R 6250 5900 50
-F26 "GPIO8-cpu" I R 6250 6000 50
-F27 "TRIG1-cpu" I L 4950 5200 50
-F28 "TRIG2-cpu" I L 4950 5300 50
-F29 "CAN2RX-cpu" I L 4950 5400 50
-F30 "CAN2TX-cpu" I L 4950 5500 50
-F31 "FREQ1-cpu" I L 4950 5600 50
-F32 "FREQ2-cpu" I L 4950 5700 50
-F33 "FREQ3-cpu" I L 4950 5800 50
-F34 "PWM1-cpu" I L 4950 5900 50
-F35 "PWM2-cpu" I L 4950 6000 50
-F36 "PWM3-cpu" I L 4950 6100 50
-F37 "PWM4-cpu" I L 4950 6200 50
-F38 "CS-cpu" I L 4950 6450 50
-F39 "SCK-cpu" I L 4950 6550 50
-F40 "MISO-cpu" I L 4950 6650 50
-F41 "MOSI-cpu" I L 4950 6750 50
-F42 "5v_cpu" I L 4950 4050 50
-F43 "CANH" I R 6250 6300 50
-F44 "CANL" I R 6250 6400 50
+F2 "IG1-cpu" I R 6250 3700 50
+F3 "IG2-cpu" I R 6250 3800 50
+F4 "IG3-cpu" I R 6250 3900 50
+F5 "IG4-cpu" I R 6250 4000 50
+F6 "INJ1-cpu" I R 6250 4100 50
+F7 "INJ2-cpu" I R 6250 4200 50
+F8 "INJ3-cpu" I R 6250 4300 50
+F9 "INJ4-cpu" I R 6250 4400 50
+F10 "INJ5-cpu" I R 6250 4500 50
+F11 "INJ6-cpu" I R 6250 4600 50
+F12 "OUT1-cpu" I R 6250 4700 50
+F13 "OUT2-cpu" I R 6250 4800 50
+F14 "OUT3-cpu" I R 6250 4900 50
+F15 "OUT4-cpu" I R 6250 5000 50
+F16 "OUT5-cpu" I R 6250 5100 50
+F17 "OUT6-cpu" I R 6250 5200 50
+F18 "GPIO1-cpu" I R 6250 5300 50
+F19 "GPIO2-cpu" I R 6250 5400 50
+F20 "GPIO3-cpu" I R 6250 5500 50
+F21 "GPIO4-cpu" I R 6250 5600 50
+F22 "GPIO5-cpu" I R 6250 5700 50
+F23 "GPIO6-cpu" I R 6250 5800 50
+F24 "GPIO7-cpu" I R 6250 5900 50
+F25 "GPIO8-cpu" I R 6250 6000 50
+F26 "TRIG1-cpu" I L 4950 5200 50
+F27 "TRIG2-cpu" I L 4950 5300 50
+F28 "CAN2RX-cpu" I L 4950 5400 50
+F29 "CAN2TX-cpu" I L 4950 5500 50
+F30 "FREQ1-cpu" I L 4950 5600 50
+F31 "FREQ2-cpu" I L 4950 5700 50
+F32 "FREQ3-cpu" I L 4950 5800 50
+F33 "PWM1-cpu" I L 4950 5900 50
+F34 "PWM2-cpu" I L 4950 6000 50
+F35 "PWM3-cpu" I L 4950 6100 50
+F36 "PWM4-cpu" I L 4950 6200 50
+F37 "CS-cpu" I L 4950 6450 50
+F38 "SCK-cpu" I L 4950 6550 50
+F39 "MISO-cpu" I L 4950 6650 50
+F40 "MOSI-cpu" I L 4950 6750 50
+F41 "5v_cpu" I L 4950 4050 50
+F42 "CANH" I R 6250 6300 50
+F43 "CANL" I R 6250 6400 50
 $EndSheet
 Wire Wire Line
@@
 Wire Wire Line
 	8150 4300 8300 4300
-$Comp
-L Connector_Generic:Conn_01x06 J7
-U 1 1 5BFE8476
-P 6650 4900
-F 0 "J7" H 6730 4846 50  0000 L CNN
-F 1 "Conn_01x06" H 6730 4801 50  0001 L CNN
-F 2 "Connector_PinHeader_2.54mm:PinHeader_1x06_P2.54mm_Vertical" H 6650 4900 50  0001 C CNN
-F 3 "~" H 6650 4900 50  0001 C CNN
-	1    6650 4900
-	1    0    0    -1
-$EndComp
 $Comp
 L Connector_Generic:Conn_01x04 J8
@@
 Text Label 4100 4050 2    50   ~ 0
 5v_cpu
-$Comp
-L Device:Jumper JP1
-U 1 1 5C011FB5
-P 4550 3750
-F 0 "JP1" H 4550 4014 50  0000 C CNN
-F 1 "Jumper" H 4550 3923 50  0000 C CNN
-F 2 "Connector_PinHeader_2.54mm:PinHeader_1x02_P2.54mm_Vertical" H 4550 3750 50  0001 C CNN
-F 3 "~" H 4550 3750 50  0001 C CNN
-	1    4550 3750
-	1    0    0    -1
-$EndComp
 Wire Wire Line
 	4100 4050 4250 4050
-Wire Wire Line
-	4850 3750 4950 3750
-Wire Wire Line
-	4250 3750 4250 4050
 Connection ~ 4250 4050
 Wire Wire Line
@@
 Wire Wire Line
 	2000 5100 1650 5100
+$Comp
+L Connector_Generic:Conn_01x04 J7
+U 1 1 5C1475FB
+P 6650 4800
+F 0 "J7" H 6730 4792 50  0000 L CNN
+F 1 "Conn_01x04" H 6730 4701 50  0000 L CNN
+F 2 "Connector_PinHeader_2.54mm:PinHeader_1x04_P2.54mm_Vertical" H 6650 4800 50  0001 C CNN
+F 3 "~" H 6650 4800 50  0001 C CNN
+	1    6650 4800
+	1    0    0    -1
+$EndComp
+$Comp
+L Connector_Generic:Conn_01x02 J21
+U 1 1 5C14774C
+P 6650 5100
+F 0 "J21" H 6730 5092 50  0000 L CNN
+F 1 "Conn_01x02" H 6730 5001 50  0000 L CNN
+F 2 "Connector_PinHeader_2.54mm:PinHeader_1x02_P2.54mm_Vertical" H 6650 5100 50  0001 C CNN
+F 3 "~" H 6650 5100 50  0001 C CNN
+	1    6650 5100
+	1    0    0    -1
+$EndComp
+Entry Bus Bus
+	1400 4300 1500 4400
 $EndSCHEMATC

Commit message: Misc fixes
Parts:
- C1: Digikey-Part 445-14799-1-ND -> 445-8034-1-ND
- C2, C3: Digikey-Part (none) -> 478-10836-1-ND
- J1: Digikey-Part (none) -> 609-3220-ND
- J10, J4, J7, J8: Digikey-Part (none) -> 732-5317-ND
- J11, J9: Digikey-Part (none) -> 732-5321-ND
- J12, J2, J21, J5, J6: Digikey-Part (none) -> 952-2262-ND
- J13, J14: Digikey-Part (none) -> 732-5319-ND
- J15: Digikey-Part (none) -> 732-5297-ND
- J3: Digikey-Part (none) -> 732-5316-ND
- R1, R2, R3, R4: Digikey-Part (none) -> P100KDACT-ND
- U1: Digikey-Part (none) -> LM2940T-5.0/NOPB-ND
