File: io.sch (KiCad schematic (older format))
At the start: 98 parts, among them P1 CONN_01X04, P2 CONN_01X04, P3 CONN_01X04, P4 CONN_02X06, P5 CONN_02X09, Q1 VND7NV04, Q2 VND7NV04, Q3 VND7NV04, Q4 VND7NV04, Q5 VND7NV04, Q6 VND7NV04, U1 TC4427, U2 TC4427, U3 TC4427, U4 MCP2562-H/P, U5 LM2940

Commit message: Add notes and ratings
Parts:
- C6: Rating (none) -> Tantalum 35V
- C7, C8: Rating (none) -> X7R
- C9: Rating (none) -> Tantalum 10V
- D11, D12, D2, D3: Notes (none) -> Schottky
- U1: value TC4427 -> TC4424
Changed lines of the file:
@@
 F 2 "Capacitors_ThroughHole:C_Disc_D3_P2.5" H 4388 800 50  0001 C CNN
 F 3 "" H 4350 950 50  0000 C CNN
+F 4 "X7R" H 4350 950 60  0001 C CNN "Rating"
 	1    4350 950
 	1    0    0    -1
@@
 F 2 "Capacitors_ThroughHole:C_Disc_D3_P2.5" H 4138 800 50  0001 C CNN
 F 3 "" H 4100 950 50  0000 C CNN
+F 4 "Tantalum 35V" H 4100 950 60  0001 C CNN "Rating"
 	1    4100 950
 	1    0    0    -1
@@
 F 2 "Capacitors_ThroughHole:C_Disc_D3_P2.5" H 5438 800 50  0001 C CNN
 F 3 "" H 5400 950 50  0000 C CNN
+F 4 "X7R" H 5400 950 60  0001 C CNN "Rating"
 	1    5400 950
 	1    0    0    -1
@@
 F 2 "Capacitors_ThroughHole:C_Disc_D3_P2.5" H 5738 800 50  0001 C CNN
 F 3 "" H 5700 950 50  0000 C CNN
+F 4 "Tantalum 10V" H 5700 950 60  0001 C CNN "Rating"
 	1    5700 950
 	1    0    0    -1
@@
 P 2250 6800
 F 0 "U1" H 2250 7050 60  0000 C CNN
-F 1 "TC4427" H 2400 6550 50  0000 C CNN
+F 1 "TC4424" H 2400 6550 50  0000 C CNN
 F 2 "Housings_DIP:DIP-8_W7.62mm" H 2250 6800 60  0001 C CNN
 F 3 "" H 2250 6800 60  0000 C CNN
@@
 F 2 "Diodes_ThroughHole:Diode_DO-41_SOD81_Vertical_KathodeUp" H 2350 10050 50  0001 C CNN
 F 3 "" H 2350 10050 50  0000 C CNN
+F 4 "Schottky" H 2350 10050 60  0001 C CNN "Notes"
 	1    2350 10050
 	0    1    1    0
@@
 F 2 "Diodes_ThroughHole:Diode_DO-41_SOD81_Vertical_KathodeUp" H 2350 10350 50  0001 C CNN
 F 3 "" H 2350 10350 50  0000 C CNN
+F 4 "Schottky" H 2350 10350 60  0001 C CNN "Notes"
 	1    2350 10350
 	0    1    1    0
@@
 F 2 "Diodes_ThroughHole:Diode_DO-41_SOD81_Vertical_KathodeUp" H 5150 10050 50  0001 C CNN
 F 3 "" H 5150 10050 50  0000 C CNN
+F 4 "Schottky" H 5150 10050 60  0001 C CNN "Notes"
 	1    5150 10050
 	0    1    1    0
@@
 F 2 "Diodes_ThroughHole:Diode_DO-41_SOD81_Vertical_KathodeUp" H 5150 10350 50  0001 C CNN
 F 3 "" H 5150 10350 50  0000 C CNN
+F 4 "Schottky" H 5150 10350 60  0001 C CNN "Notes"
 	1    5150 10350
 	0    1    1    0

Commit message: Various updates to io board: - Add trigger inputs - Switch to 3v logic fets - switch to SMT components
Parts:
- removed C1, C2: 0.1 uF, Capacitors_ThroughHole:C_Disc_D3_P2.5, symbol C
- removed C4, C5: 1 uF, Capacitors_ThroughHole:C_Disc_D3_P2.5, symbol C
- removed D1: 3.3 V Zener, Diodes_ThroughHole:Diode_DO-41_SOD81_Vertical_KathodeUp, symbol D_Zener
- removed D10, D13, D14, D15, D16, D17, D18, D5, D6, D7, D8, D9: LED, LEDs:LED-3MM, symbol LED
- removed D11, D12, D2, D20, D21, D22, D23, D24, D25, D26, D27, D3: D, Diodes_ThroughHole:Diode_DO-41_SOD81_Vertical_KathodeUp, symbol D
- removed D19, D4: D_Zener, Diodes_ThroughHole:Diode_DO-41_SOD81_Vertical_KathodeUp, symbol D_Zener
- removed P1: CONN_01X04, Pin_Headers:Pin_Header_Straight_1x04, symbol CONN_01X04
- removed P4: CONN_02X06, Pin_Headers:Pin_Header_Straight_2x06, symbol CONN_02X06
- removed P5: CONN_02X09, Pin_Headers:Pin_Header_Straight_2x09, symbol CONN_02X09
- removed Q1, Q2, Q3, Q4, Q5, Q6: VND7NV04, TO_SOT_Packages_SMD:TO-252-2Lead, symbol VND14NV04
- removed R1, R2, R29, R3, R48, R5, R6, R7: 1k, Resistors_ThroughHole:Resistor_Horizontal_RM7mm, symbol R
- removed R11, R12, R13, R34, R35, R36, R37, R40, R41, R8, R9: 100k, Resistors_ThroughHole:Resistor_Horizontal_RM7mm, symbol R
- removed R18, R19, R20: 150, Resistors_ThroughHole:Resistor_Horizontal_RM7mm, symbol R
- removed R22, R23, R25, R26, R27, R28, R30, R31, R32, R33, R38, R39: 2.43k, Resistors_ThroughHole:Resistor_Horizontal_RM7mm, symbol R
- removed R24: 120, Resistors_ThroughHole:Resistor_Horizontal_RM7mm, symbol R
- removed R43, R44, R45, R46, R47: 330, Resistors_ThroughHole:Resistor_Horizontal_RM7mm, symbol R
- removed U1: TC4424, Housings_DIP:DIP-8_W7.62mm, symbol TC4427
- removed U2, U3: TC4427, Housings_DIP:DIP-8_W7.62mm, symbol TC4427
- removed U4: MCP2562-H/P, Housings_DIP:DIP-8_W7.62mm, symbol MCP2562-H/P
- added C10, C11, C12, C13, C15, C16, C17, C18: .1uF, Capacitor_SMD:C_0805_2012Metric_Pad1.18x1.45mm_HandSolder, symbol analog-rescue:C
- added C14: 1u, Capacitor_SMD:C_0805_2012Metric_Pad1.18x1.45mm_HandSolder, symbol analog-rescue:C
- added C19, C20: 1 uF, Capacitor_SMD:C_0805_2012Metric_Pad1.18x1.45mm_HandSolder, symbol io-rescue:C-io-rescue
- added C6, C7: 1n, Capacitor_SMD:C_0805_2012Metric_Pad1.18x1.45mm_HandSolder, symbol analog-rescue:C
- added C8: 10n, Capacitor_SMD:C_0805_2012Metric_Pad1.18x1.45mm_HandSolder, symbol analog-rescue:C
- added C9: 0.1u, Capacitor_SMD:C_0805_2012Metric_Pad1.18x1.45mm_HandSolder, symbol analog-rescue:C
- added D1, D2: BAT54S, Package_TO_SOT_SMD:SOT-23, symbol Diode:BAT54S
- added JP1: IG_PWR, Jumper:SolderJumper-3_P1.3mm_Open_Pad1.0x1.5mm, symbol Jumper:SolderJumper_3_Open
- added P1: OUT_GND, Connector_PinHeader_2.54mm:PinHeader_1x04_P2.54mm_Horizontal, symbol io-rescue:CONN_01X04-io-rescue
- added P10: INJ-CPU, Connector_PinHeader_2.54mm:PinHeader_1x04_P2.54mm_Horizontal, symbol io-rescue:CONN_01X04-io-rescue
- added P12: LSD-CPU, Connector_PinHeader_2.54mm:PinHeader_1x04_P2.54mm_Horizontal, symbol io-rescue:CONN_01X04-io-rescue
- added P2: TRIG-cpu, Connector_PinHeader_2.54mm:PinHeader_1x04_P2.54mm_Horizontal, symbol io-rescue:CONN_01X04-io-rescue
- added P3: DIG-CPU, Connector_PinHeader_2.54mm:PinHeader_1x04_P2.54mm_Horizontal, symbol io-rescue:CONN_01X04-io-rescue
- added P4: IN-CPU, Connector_PinHeader_2.54mm:PinHeader_1x04_P2.54mm_Horizontal, symbol io-rescue:CONN_01X04-io-rescue
- added P5: CPU_PWR, Connector_PinHeader_2.54mm:PinHeader_1x04_P2.54mm_Horizontal, symbol io-rescue:CONN_01X04-io-rescue
- added P6: TRIG-IN, Connector_PinHeader_2.54mm:PinHeader_1x04_P2.54mm_Horizontal, symbol io-rescue:CONN_01X04-io-rescue
- added P7: DIG-IN, Connector_PinHeader_2.54mm:PinHeader_1x04_P2.54mm_Horizontal, symbol io-rescue:CONN_01X04-io-rescue
- added P8: IGNITION, Connector_PinHeader_2.54mm:PinHeader_1x04_P2.54mm_Horizontal, symbol io-rescue:CONN_01X04-io-rescue
- added P9: PWR_IN, Connector_PinHeader_2.54mm:PinHeader_1x04_P2.54mm_Horizontal, symbol io-rescue:CONN_01X04-io-rescue
- added Q1, Q2, Q3, Q4, Q5, Q6, Q7, Q8: MOSFET, Package_TO_SOT_SMD:TO-252-2, symbol io-rescue:VND14NV04-io-rescue
- added R1, R2, R21, R22, R23, R24: 1k, Resistor_SMD:R_0805_2012Metric_Pad1.20x1.40mm_HandSolder, symbol analog-rescue:R
- added R10, R7: 10k, Resistor_SMD:R_0805_2012Metric_Pad1.20x1.40mm_HandSolder, symbol analog-rescue:R
- added R11, R17, R41, R42, R43, R44, R45, R46, R47, R48, R9: 100k, Resistor_SMD:R_0805_2012Metric_Pad1.20x1.40mm_HandSolder, symbol io-rescue:R-io-rescue
- added R14, R15, R16: 150, Resistor_SMD:R_0805_2012Metric_Pad1.20x1.40mm_HandSolder, symbol io-rescue:R-io-rescue
- added R18, R19, R20, R27, R28, R29, R31, R32, R33, R34, R35, R36, R37, R38, R39, R4, R40, R49, R5, R50: 1k, Resistor_SMD:R_0805_2012Metric_Pad1.20x1.40mm_HandSolder, symbol io-rescue:R-io-rescue
- added R25, R26: 330, Resistor_THT:R_Axial_DIN0207_L6.3mm_D2.5mm_P2.54mm_Vertical, symbol analog-rescue:R
- added R51, R52, R53, R54, R55, R56, R57, R58: 100k, Resistor_SMD:R_0805_2012Metric_Pad1.20x1.40mm_HandSolder, symbol analog-rescue:R
- added U10, U11, U4, U5, U6, U7, U8, U9: BTF3080EJ, Package_SO:Infineon_PG-DSO-8-27_3.9x4.9mm_EP2.65x3mm, symbol io-rescue:BTF3080EJ
- added U12, U13, U2: MIC4469, Package_SO:SOIC-16W_7.5x10.3mm_P1.27mm, symbol io-rescue:MIC4469-viaems
- added U3: MAX9926UAEE+, Package_SO:QSOP-16_3.9x4.9mm_P0.635mm, symbol viaems:MAX9926UAEE+
- C1: renamed from C6; footprint Capacitors_ThroughHole:C_Disc_D3_P2.5 -> Capacitor_SMD:C_0805_2012Metric_Pad1.18x1.45mm_HandSolder; symbol C -> io-rescue:C-io-rescue
- C2: renamed from C7; footprint Capacitors_ThroughHole:C_Disc_D3_P2.5 -> Capacitor_SMD:C_0805_2012Metric_Pad1.18x1.45mm_HandSolder; symbol C -> io-rescue:C-io-rescue
- C3: renamed from C8; footprint Capacitors_ThroughHole:C_Disc_D3_P2.5 -> Capacitor_SMD:C_0805_2012Metric_Pad1.18x1.45mm_HandSolder; symbol C -> io-rescue:C-io-rescue
- C4: renamed from C9; footprint Capacitors_ThroughHole:C_Disc_D3_P2.5 -> Capacitor_SMD:C_1206_3216Metric; symbol C -> io-rescue:C-io-rescue
- C5: renamed from C3; footprint Capacitors_ThroughHole:C_Disc_D3_P2.5 -> Capacitor_SMD:C_0805_2012Metric_Pad1.18x1.45mm_HandSolder; symbol C -> io-rescue:C-io-rescue
- P11: renamed from P2; value CONN_01X04 -> INJECTORS; footprint Pin_Headers:Pin_Header_Straight_1x04 -> Connector_PinHeader_2.54mm:PinHeader_1x04_P2.54mm_Horizontal; symbol CONN_01X04 -> io-rescue:CONN_01X04-io-rescue
- P13: renamed from P3; value CONN_01X04 -> LSDS; footprint Pin_Headers:Pin_Header_Straight_1x04 -> Connector_PinHeader_2.54mm:PinHeader_1x04_P2.54mm_Horizontal; symbol CONN_01X04 -> io-rescue:CONN_01X04-io-rescue
- R12: renamed from R21; footprint Resistors_ThroughHole:Resistor_Horizontal_RM7mm -> Resistor_SMD:R_0805_2012Metric_Pad1.20x1.40mm_HandSolder; symbol R -> io-rescue:R-io-rescue
- R13: renamed from R17; footprint Resistors_ThroughHole:Resistor_Horizontal_RM7mm -> Resistor_SMD:R_0805_2012Metric_Pad1.20x1.40mm_HandSolder; symbol R -> io-rescue:R-io-rescue
- R3: renamed from R4; footprint Resistors_ThroughHole:Resistor_Horizontal_RM7mm -> Resistor_SMD:R_0805_2012Metric_Pad1.20x1.40mm_HandSolder; symbol R -> io-rescue:R-io-rescue
- R30: renamed from R42; value 330 -> 1k; footprint Resistors_ThroughHole:Resistor_Horizontal_RM7mm -> Resistor_SMD:R_0805_2012Metric_Pad1.20x1.40mm_HandSolder; symbol R -> io-rescue:R-io-rescue
- R6: renamed from R10; footprint Resistors_ThroughHole:Resistor_Horizontal_RM7mm -> Resistor_SMD:R_0805_2012Metric_Pad1.20x1.40mm_HandSolder; symbol R -> io-rescue:R-io-rescue
- R8: renamed from R14; footprint Resistors_ThroughHole:Resistor_Horizontal_RM7mm -> Resistor_SMD:R_0805_2012Metric_Pad1.20x1.40mm_HandSolder; symbol R -> io-rescue:R-io-rescue
- U1: renamed from U5; footprint TO_SOT_Packages_THT:TO-220_Neutral123_Horizontal_LargePads -> Package_TO_SOT_THT:TO-220-3_Horizontal_TabDown; symbol LM2940 -> io-rescue:LM2940-io-rescue
Connections:
- net 12v_power: now also JP1.1 (A), P7.4 (P4), P9.1 (P1), P9.2 (P2); no longer C5.1
- net DIG1-cpu: now also P3.2 (P2)
- net DIG1-in: now also P7.2 (P2)
- net DIG2-cpu: now also P3.3 (P3), R18.2
- net DIG2-in: now also P7.3 (P3), R20.1
- net GND: now also C14.2, C19.2, C20.2, C8.2, C9.2, D1.1, D2.1, P2.4 (P4), P3.1 (P1), P5.3 (P3), P5.4 (P4), P7.1 (P1), P9.3 (P3), P9.4 (P4), R11.1, R17.1, R41.1, R42.1, R43.1, R44.1, R45.1, R46.1, R47.1, R48.1, R9.1, U12.10 (4B), U12.2 (1B), U12.4 (2B), U12.6 (3B), U12.7 (GND), U12.8 (GND), U13.10 (4B), U13.2 (1B), U13.4 (2B), U13.6 (3B), U13.7 (GND), U13.8 (GND), U2.10 (4B), U2.2 (1B), U2.4 (2B), U2.6 (3B), U2.7 (GND), U2.8 (GND), U3.1 (INT_THRS1), U3.11 (GND), U3.13 (ZERO_EN), U3.3 (BIAS1), U3.6 (BIAS2), U3.8 (IN_THRS2)
- net IG1-cpu: now also P4.1 (P1)
- net IG1-out: now also P8.1 (P1)
- net IG2-cpu: now also P4.2 (P2), R4.2
- net IG2-out: now also P8.2 (P2), R14.1
- net IG3-cpu: now also P4.3 (P3), R5.2
- net IG3-out: now also P8.3 (P3), R15.1
- net IG4-cpu: now also P4.4 (P4), R19.2
- net IG4-out: now also P8.4 (P4), R16.1
- net INJ1-cpu: now also P10.4 (P4), R35.2
- net INJ1-out: now also Q1.2 (D), U7.9 (OUT)
- net INJ2-cpu: now also P10.3 (P3), R28.2, R36.2
- net INJ2-out: now also P11.2 (P2), Q3.2 (D), U5.9 (OUT); no longer P11.3 (P3)
- net INJ3-cpu: now also P10.2 (P2), R29.2, R37.2
- net INJ3-out: now also P11.3 (P3), Q5.2 (D), U6.9 (OUT); no longer P13.1 (P1)
- net INJ4-cpu: now also P10.1 (P1), R27.2, R49.2
- net INJ4-out: now also P11.4 (P4), Q7.2 (D), U4.9 (OUT); no longer P13.3 (P3)
- net LSD1-cpu: now also P12.4 (P4), R34.2, R38.2, R39.2
- net LSD1-out: now also P13.1 (P1), Q2.2 (D), U11.9 (OUT)
- net LSD2-cpu: now also P12.3 (P3), R32.2
- net LSD2-out: now also P13.2 (P2), Q4.2 (D), U9.9 (OUT)
- net OUT_GND: now also C10.2, C11.2, C12.2, C13.2, C15.2, C16.2, C17.2, C18.2, P1.1 (P1), P1.2 (P2), P1.3 (P3), P1.4 (P4), Q1.3 (S), Q2.3 (S), Q3.3 (S), Q4.3 (S), Q5.3 (S), Q6.3 (S), Q7.3 (S), Q8.3 (S), R51.2, R52.2, R53.2, R54.2, R55.2, R56.2, R57.2, R58.2, U10.4 (SRP), U10.6 (GND), U10.7 (GND), U10.8 (GND), U11.4 (SRP), U11.6 (GND), U11.7 (GND), U11.8 (GND), U4.4 (SRP), U4.6 (GND), U4.7 (GND), U4.8 (GND), U5.4 (SRP), U5.6 (GND), U5.7 (GND), U5.8 (GND), U6.4 (SRP), U6.6 (GND), U6.7 (GND), U6.8 (GND), U7.4 (SRP), U7.6 (GND), U7.7 (GND), U7.8 (GND), U8.4 (SRP), U8.6 (GND), U8.7 (GND), U8.8 (GND), U9.4 (SRP), U9.6 (GND), U9.7 (GND), U9.8 (GND); no longer P11.2 (P2), P11.4 (P4), P13.2 (P2), P13.4 (P4)
- net at R30.1: now also U7.1 (IN)
- net at R6.2: now also R5.1, U2.5 (3A); no longer R3.1
- net at R13.2: now also U2.14 (1Y)
- net at R12.2, R8.1: now also D1.3
- net 5v_cpu renamed 5v
- net 5v: now also C10.1, C11.1, C12.1, C13.1, C14.1, C15.1, C16.1, C17.1, C18.1, C19.1, C20.1, C8.1, C9.1, D1.2, D2.2, JP1.3 (B), P2.1 (P1), P3.4 (P4), P5.1 (P1), P5.2 (P2), R10.1, R7.1, U10.2 (Vdd), U10.5 (ENABLE), U11.2 (Vdd), U11.5 (ENABLE), U12.15 (Vs), U12.16 (Vs), U13.15 (Vs), U13.16 (Vs), U3.14 (VCC), U4.2 (Vdd), U4.5 (ENABLE), U5.2 (Vdd), U5.5 (ENABLE), U6.2 (Vdd), U6.5 (ENABLE), U7.2 (Vdd), U7.5 (ENABLE), U8.2 (Vdd), U8.5 (ENABLE), U9.2 (Vdd), U9.5 (ENABLE)
- new net: R11.2, R3.1, U2.1 (1A)
- new net: C5.1, JP1.2 (C), U2.15 (Vs), U2.16 (Vs)
- new net: R16.2, U2.11 (4Y)
- new net: R15.2, U2.12 (3Y)
- new net: R14.2, U2.13 (2Y)
- new net: R4.1, R9.2, U2.3 (2A)
- new net: R17.2, R19.1, U2.9 (4A)
- new net: R37.1, R41.2, U12.5 (3A)
- new net: R35.1, R45.2, U12.1 (1A)
- new net: Q7.1 (G), R57.1, U12.11 (4Y)
- new net: Q5.1 (G), R55.1, U12.12 (3Y)
- new net: Q3.1 (G), R53.1, U12.13 (2Y)
- new net: Q1.1 (G), R51.1, U12.14 (1Y)
- new net: R36.1, R43.2, U12.3 (2A)
- new net: R47.2, R49.1, U12.9 (4A)
- new net: R28.1, U5.1 (IN)
- new net: R29.1, U6.1 (IN)
- new net: R27.1, U4.1 (IN)
- new net: Q8.1 (G), R58.1, U13.11 (4Y)
- new net: Q6.1 (G), R56.1, U13.12 (3Y)
- new net: Q4.1 (G), R54.1, U13.13 (2Y)
- new net: Q2.1 (G), R52.1, U13.14 (1Y)
- new net: R48.2, R50.1, U13.9 (4A)
- new net: R38.1, R46.2, U13.1 (1A)
- new net: R39.1, R44.2, U13.3 (2A)
- new net: R40.1, R42.2, U13.5 (3A)
- new net: R34.1, U11.1 (IN)
- new net: R32.1, U9.1 (IN)
- new net: R33.1, U10.1 (IN)
- new net: R31.1, U8.1 (IN)
- new net: C7.1, R23.2, U3.10 (IN2-)
- new net: C6.2, R22.2, U3.15 (IN1-)
- new net: C6.1, R21.2, U3.16 (IN1+)
- new net: R1.1, R10.2, U3.4 (COUT1)
- new net: R2.1, R7.2, U3.5 (COUT2)
- new net: C7.2, R24.2, U3.9 (IN2+)
- new net: D2.3, R18.1, R20.2
- new net LSD3-cpu: P12.2 (P2), R33.2, R40.2
- new net LSD3-out: P13.3 (P3), Q6.2 (D), U10.9 (OUT)
- new net LSD4-cpu: P12.1 (P1), R31.2, R50.2
- new net LSD4-out: P13.4 (P4), Q8.2 (D), U8.9 (OUT)
- new net TRIG1: P2.3 (P3), R1.2
- new net TRIG1IN+: P6.2 (P2), R21.1, R25.1
- new net TRIG1IN-: P6.1 (P1), R22.1, R25.2
- new net TRIG2: P2.2 (P2), R2.2
- new net TRIG2IN+: P6.4 (P4), R24.1, R26.2
- new net TRIG2IN-: P6.3 (P3), R23.1, R26.1
- no-connect marks 6 -> 11
Other:
- note added: "Fuel and Lowside Driver alternative\nOnly either populate if above drivers not populated. Use this as an alternative to use standard TO-252 N-channel mosfets with a dedicated gate driver."
- note added: "Low Side Drivers"
- note added: "Trigger Inputs"
- note removed: "CANBUS"
- note removed: "High-Side Drivers"
- note removed: "IO"
- note removed: "Low-Side Drivers"
- moved on the sheet: C1, C2, C3, C4, C5, P11, P13, R12, R13, R3, R30, R6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
