File: analog.sch (KiCad schematic (older format))
At the start: 63 parts, among them P1 CONN_01X09, P2 CONN_01X06, P3 CONN_01X06, P4 CONN_01X05, U1 LM2940, U2 TLC2543

Commit message: fixups
Parts:
- removed C10, C13, C14, C15, C19, C2, C3, C9: 0.1 uF, Capacitors_ThroughHole:C_Disc_D3_P2.5, symbol C
- removed C18, C20: 10 uF, Capacitors_ThroughHole:C_Disc_D3_P2.5, symbol C
- removed C21, C22, C23, C24, C25: 0.47 uF, Capacitors_ThroughHole:C_Disc_D3_P2.5, symbol C
- removed D1, D10, D11, D12, D2, D3, D4, D5, D6, D7, D8, D9: 1N5818, Diodes_ThroughHole:Diode_DO-41_SOD81_Vertical_KathodeUp, symbol D_Schottky
- removed P1: CONN_01X09, Pin_Headers:Pin_Header_Straight_1x09, symbol CONN_01X09
- removed P2: CONN_01X06, Pin_Headers:Pin_Header_Straight_1x06, symbol CONN_01X06
- removed P4: CONN_01X05, Pin_Headers:Pin_Header_Straight_1x05, symbol CONN_01X05
- removed R12: 100, Resistors_ThroughHole:Resistor_Horizontal_RM7mm, symbol R
- removed R9: 2.49k, Resistors_ThroughHole:Resistor_Horizontal_RM7mm, symbol R
- removed U2: TLC2543, Housings_DIP:DIP-20_W7.62mm, symbol TLC2543
- added C10, C12, C13, C17, C25, C5, C7, C9: 0.1 uF, Capacitor_SMD:C_0805_2012Metric_Pad1.18x1.45mm_HandSolder, symbol analog-rescue:C
- added C14, C18, C22, C23, C26, C27, C28, C29: 0.47 uF, Capacitor_SMD:C_0805_2012Metric_Pad1.18x1.45mm_HandSolder, symbol analog-rescue:C
- added C16: 1 uF, Capacitor_SMD:C_0805_2012Metric_Pad1.18x1.45mm_HandSolder, symbol analog-rescue:C
- added C20: 0.01 uF, Capacitor_SMD:C_0805_2012Metric_Pad1.18x1.45mm_HandSolder, symbol analog-rescue:C
- added C24: 0.33 uF, Capacitor_SMD:C_0805_2012Metric_Pad1.18x1.45mm_HandSolder, symbol analog-rescue:C
- added D1, D10, D11, D12, D13, D14, D2, D3, D5, D6, D7, D8, D9: BAT54S, Package_TO_SOT_SMD:SOT-23, symbol Diode:BAT54S
- added D4: 5.4 V, Diode_THT:D_A-405_P2.54mm_Vertical_AnodeUp, symbol Device:D_Zener
- added F1: 500 mA, Fuse:Fuse_1206_3216Metric_Pad1.42x1.75mm_HandSolder, symbol Device:Polyfuse
- added J1: SPARE1, Connector_PinHeader_2.54mm:PinHeader_1x04_P2.54mm_Horizontal, symbol Connector_Generic:Conn_01x04
- added J2: SPARE2, Connector_PinHeader_2.54mm:PinHeader_1x04_P2.54mm_Horizontal, symbol Connector_Generic:Conn_01x04
- added J3: MAIN, Connector_PinHeader_2.54mm:PinHeader_1x04_P2.54mm_Horizontal, symbol Connector_Generic:Conn_01x04
- added J4: KNOCK, Connector_PinHeader_2.54mm:PinHeader_1x04_P2.54mm_Horizontal, symbol Connector_Generic:Conn_01x04
- added J5: POWER, Connector_PinHeader_2.54mm:PinHeader_1x04_P2.54mm_Horizontal, symbol Connector_Generic:Conn_01x04
- added R10, R24, R29, R30, R31, R32, R33, R34: 220, Resistor_SMD:R_0805_2012Metric_Pad1.20x1.40mm_HandSolder, symbol analog-rescue:R
- added R12, R13: 120, Resistor_SMD:R_0805_2012Metric_Pad1.20x1.40mm_HandSolder, symbol analog-rescue:R
- added R22, R23, R6, R7: 1000, Resistor_SMD:R_0805_2012Metric_Pad1.20x1.40mm_HandSolder, symbol analog-rescue:R
- added R8, R9: 330, Resistor_SMD:R_0805_2012Metric_Pad1.20x1.40mm_HandSolder, symbol analog-rescue:R
- added U1: MAX11632, Package_SO:QSOP-24_3.9x8.7mm_P0.635mm, symbol viaems:MAX11632
- added U3: MCP6002-xSN, Package_SO:MSOP-8_3x3mm_P0.65mm, symbol Amplifier_Operational:MCP6002-xSN
- added U4: MPXA6400A, Sensor_Pressure:Freescale_98ARH99089A, symbol Sensor_Pressure:MPXA6115A
- C1: footprint Capacitors_ThroughHole:C_Disc_D3_P2.5 -> Capacitor_SMD:C_0805_2012Metric_Pad1.18x1.45mm_HandSolder; symbol C -> analog-rescue:C
- C11: value 0.47 uF -> 1 uF; footprint Capacitors_ThroughHole:C_Disc_D3_P2.5 -> Capacitor_SMD:C_0805_2012Metric_Pad1.18x1.45mm_HandSolder; symbol C -> analog-rescue:C
- C15: renamed from C6; value 0.47 uF -> 1 uF; footprint Capacitors_ThroughHole:C_Disc_D3_P2.5 -> Capacitor_SMD:C_0805_2012Metric_Pad1.18x1.45mm_HandSolder; symbol C -> analog-rescue:C
- C19: renamed from C17; value 0.47 uF -> 1 uF; footprint Capacitors_ThroughHole:C_Disc_D3_P2.5 -> Capacitor_SMD:C_0805_2012Metric_Pad1.18x1.45mm_HandSolder; symbol C -> analog-rescue:C
- C2: renamed from C12; footprint Capacitors_ThroughHole:C_Disc_D3_P2.5 -> Capacitor_SMD:C_0805_2012Metric_Pad1.18x1.45mm_HandSolder; symbol C -> analog-rescue:C
- C21: renamed from C16; footprint Capacitors_ThroughHole:C_Disc_D3_P2.5 -> Capacitor_SMD:C_0805_2012Metric_Pad1.18x1.45mm_HandSolder; symbol C -> analog-rescue:C
- C3: renamed from C4; footprint Capacitors_ThroughHole:C_Disc_D3_P2.5 -> Capacitor_SMD:C_0805_2012Metric_Pad1.18x1.45mm_HandSolder; symbol C -> analog-rescue:C
- C4: renamed from C5; value 0.47 uF -> 1 uF; footprint Capacitors_ThroughHole:C_Disc_D3_P2.5 -> Capacitor_SMD:C_0805_2012Metric_Pad1.18x1.45mm_HandSolder; symbol C -> analog-rescue:C
- C6: renamed from C7; footprint Capacitors_ThroughHole:C_Disc_D3_P2.5 -> Capacitor_SMD:C_0805_2012Metric_Pad1.18x1.45mm_HandSolder; symbol C -> analog-rescue:C
- C8: footprint Capacitors_ThroughHole:C_Disc_D3_P2.5 -> Capacitor_SMD:C_1206_3216Metric_Pad1.33x1.80mm_HandSolder; symbol C -> analog-rescue:C
- P1: renamed from P3; footprint Pin_Headers:Pin_Header_Straight_1x06 -> Connector_PinHeader_2.54mm:PinHeader_1x06_P2.54mm_Horizontal; symbol CONN_01X06 -> analog-rescue:CONN_01X06
- R1: renamed from R6; value 470 -> 220; footprint Resistors_ThroughHole:Resistor_Horizontal_RM7mm -> Resistor_SMD:R_0805_2012Metric_Pad1.20x1.40mm_HandSolder; symbol R -> analog-rescue:R
- R11: renamed from R3; value 470 -> 220; footprint Resistors_ThroughHole:Resistor_Horizontal_RM7mm -> Resistor_SMD:R_0805_2012Metric_Pad1.20x1.40mm_HandSolder; symbol R -> analog-rescue:R
- R14: renamed from R13; footprint Resistors_ThroughHole:Resistor_Horizontal_RM7mm -> Resistor_SMD:R_0805_2012Metric_Pad1.20x1.40mm_HandSolder; symbol R -> analog-rescue:R
- R15: renamed from R14; footprint Resistors_ThroughHole:Resistor_Horizontal_RM7mm -> Resistor_SMD:R_0805_2012Metric_Pad1.20x1.40mm_HandSolder; symbol R -> analog-rescue:R
- R16: renamed from R15; footprint Resistors_ThroughHole:Resistor_Horizontal_RM7mm -> Resistor_SMD:R_0805_2012Metric_Pad1.20x1.40mm_HandSolder; symbol R -> analog-rescue:R
- R17: renamed from R16; footprint Resistors_ThroughHole:Resistor_Horizontal_RM7mm -> Resistor_SMD:R_0805_2012Metric_Pad1.20x1.40mm_HandSolder; symbol R -> analog-rescue:R
- R18: renamed from R17; footprint Resistors_ThroughHole:Resistor_Horizontal_RM7mm -> Resistor_SMD:R_0805_2012Metric_Pad1.20x1.40mm_HandSolder; symbol R -> analog-rescue:R
- R19: renamed from R18; footprint Resistors_ThroughHole:Resistor_Horizontal_RM7mm -> Resistor_SMD:R_0805_2012Metric_Pad1.20x1.40mm_HandSolder; symbol R -> analog-rescue:R
- R2: renamed from R1; footprint Resistors_ThroughHole:Resistor_Horizontal_RM7mm -> Resistor_SMD:R_0805_2012Metric_Pad1.20x1.40mm_HandSolder; symbol R -> analog-rescue:R
- R20: renamed from R19; footprint Resistors_ThroughHole:Resistor_Horizontal_RM7mm -> Resistor_SMD:R_0805_2012Metric_Pad1.20x1.40mm_HandSolder; symbol R -> analog-rescue:R
- R21: renamed from R20; footprint Resistors_ThroughHole:Resistor_Horizontal_RM7mm -> Resistor_SMD:R_0805_2012Metric_Pad1.20x1.40mm_HandSolder; symbol R -> analog-rescue:R
- R25: renamed from R7; footprint Resistors_ThroughHole:Resistor_Horizontal_RM7mm -> Resistor_SMD:R_0805_2012Metric_Pad1.20x1.40mm_HandSolder; symbol R -> analog-rescue:R
- R26: renamed from R8; footprint Resistors_ThroughHole:Resistor_Horizontal_RM7mm -> Resistor_SMD:R_0805_2012Metric_Pad1.20x1.40mm_HandSolder; symbol R -> analog-rescue:R
- R27: renamed from R11; value 470 -> 220; footprint Resistors_ThroughHole:Resistor_Horizontal_RM7mm -> Resistor_SMD:R_0805_2012Metric_Pad1.20x1.40mm_HandSolder; symbol R -> analog-rescue:R
- R28: renamed from R10; value 470 -> 220; footprint Resistors_ThroughHole:Resistor_Horizontal_RM7mm -> Resistor_SMD:R_0805_2012Metric_Pad1.20x1.40mm_HandSolder; symbol R -> analog-rescue:R
- R3: renamed from R2; value 470 -> 220; footprint Resistors_ThroughHole:Resistor_Horizontal_RM7mm -> Resistor_SMD:R_0805_2012Metric_Pad1.20x1.40mm_HandSolder; symbol R -> analog-rescue:R
- R4: footprint Resistors_ThroughHole:Resistor_Horizontal_RM7mm -> Resistor_SMD:R_0805_2012Metric_Pad1.20x1.40mm_HandSolder; symbol R -> analog-rescue:R
- R5: value 470 -> 220; footprint Resistors_ThroughHole:Resistor_Horizontal_RM7mm -> Resistor_SMD:R_0805_2012Metric_Pad1.20x1.40mm_HandSolder; symbol R -> analog-rescue:R
- U2: renamed from U1; footprint TO_SOT_Packages_THT:TO-220_Neutral123_Horizontal -> Package_TO_SOT_THT:TO-220-3_Horizontal_TabDown; symbol LM2940 -> analog-rescue:LM2940
Connections:
- net labels added: 2v5_knock, 5v_out, KNK1, KNK1-adc, KNK2, KNK2-adc, MAP-adc, SPR1-adc, SPR1-in, SPR2-adc, SPR2-in, SPR3-adc, SPR3-in, SPR4-adc, SPR4-in, SPR5-adc, SPR5-in, SPR6-adc, SPR6-in, SPR7-adc, SPR7-in, SPR8-adc, SPR8-in
- net labels removed: ADC_EOC, EX-1, EX-2, EX-3, EX-4, EX-5, SPR-adc, SPR-in
- wire segments 128 -> 196
- no-connect marks 0 -> 1
Other:
- moved on the sheet: C1, C11, C15, C19, C2, C21, C3, C4, C6, C8, R1, R11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
